Commit message: feat: step 2.5a — screwdriver end-effector for screw_robot
STL source: jackvial/assembler0 (packages/assembler0-hardware/stl and
assembler0-simulator assets) — option A, existing STL files used directly.

New meshes (both in mm; use scale="0.001 0.001 0.001" in URDF):
  so101_description/meshes/so101_screwdriver_bit_holder.stl  (62K)
  so101_description/meshes/screwdriver_bit.stl               (16K)

so101.urdf.xacro:
  - Added screwdriver arg (default=false)
  - Conditional <xacro:if value="$(arg screwdriver)">:
      screwdriver_tip_link  — bit_holder + bit visuals, cylinder collision
      screwdriver_tip_joint — fixed, parent gripper_link, −30mm in Z
  Gripper joint and fingers unchanged; screwdriver is additive.

so101_screwdriver.urdf.xacro (new):
  Thin wrapper that includes so101.urdf.xacro with screwdriver:=true as
  default. First-declaration-wins in xacro ensures the true default
  overrides the base file's false default.

assembly_world.launch.py:
  screw_robot spawns from so101_screwdriver.urdf.xacro (screwdriver=true).
  All other 4 arms continue using so101.urdf.xacro (screwdriver=false).

Headless verification:
  xacro output for screw_robot: screwdriver_tip_link ✓
                                 screwdriver_tip_joint ✓
                                 so101_screwdriver_bit_holder.stl ✓
                                 screwdriver_bit.stl ✓
  xacro output for lerobot_1: screwdriver_tip_link absent ✓

Co-Authored-By: Claude Sonnet 4.6 <noreply@anthropic.com>

File: so101_description/urdf/so101.urdf.xacro (robot description, xacro)
@@ -3,4 +3,6 @@
   <xacro:arg name="namespace" default=""/>
   <xacro:arg name="controllers_yaml" default="$(find so101_description)/config/ros2_controllers.yaml"/>
+  <!-- Set screwdriver:=true to add the screwdriver end-effector (used by screw_robot) -->
+  <xacro:arg name="screwdriver" default="false"/>
   <!-- Materials -->
   <material name="3d_printed">
@@ -348,3 +350,51 @@
     </plugin>
   </gazebo>
+  <!-- ============================================================
+       Screwdriver end-effector (enabled when screwdriver:=true)
+       Attaches to gripper_link; bit points in −Z of gripper_link frame.
+       Geometry (both STLs are in mm → scale 0.001):
+         bit_holder : 20mm ⌀ × 25.6mm tall, base at Z=0, tip at +Z in STL
+         screwdriver_bit : 4mm ⌀ × 43mm long
+       Both are flipped 180° (rpy π 0 0) so the tip extends in −Z.
+  ============================================================ -->
+  <xacro:if value="$(arg screwdriver)">
+    <link name="screwdriver_tip_link">
+      <inertial>
+        <origin xyz="0 0 -0.035" rpy="0 0 0"/>
+        <mass value="0.025"/>
+        <inertia ixx="1e-5" ixy="0" ixz="0" iyy="1e-5" iyz="0" izz="1e-6"/>
+      </inertial>
+      <!-- bit holder: flipped so chuck tip points in −Z -->
+      <visual>
+        <origin xyz="0 0 0" rpy="3.14159 0 0"/>
+        <geometry>
+          <mesh filename="package://so101_description/meshes/so101_screwdriver_bit_holder.stl"
+                scale="0.001 0.001 0.001"/>
+        </geometry>
+        <material name="sts3215"/>
+      </visual>
+      <!-- screwdriver bit: starts just below the holder tip -->
+      <visual>
+        <origin xyz="0 0 -0.026" rpy="3.14159 0 0"/>
+        <geometry>
+          <mesh filename="package://so101_description/meshes/screwdriver_bit.stl"
+                scale="0.001 0.001 0.001"/>
+        </geometry>
+        <material name="3d_printed"/>
+      </visual>
+      <!-- simplified collision: cylinder covering holder + bit -->
+      <collision>
+        <origin xyz="0 0 -0.035" rpy="0 0 0"/>
+        <geometry>
+          <cylinder radius="0.005" length="0.070"/>
+        </geometry>
+      </collision>
+    </link>
+    <!-- Fixed joint: 30mm below gripper_link origin, aligned with tool axis -->
+    <joint name="screwdriver_tip_joint" type="fixed">
+      <origin xyz="0 0 -0.030" rpy="0 0 0"/>
+      <parent link="gripper_link"/>
+      <child link="screwdriver_tip_link"/>
+    </joint>
+  </xacro:if>
 </robot>

Commit message: feat: step 2.5a — 2.5mm hex screwdriver tip for screw_robot
Adds a primitives-only screwdriver end-effector (shaft + taper + hex bit)
to screw_robot via so101_screwdriver.urdf.xacro; so101.urdf.xacro is
unchanged so all other arms are unaffected. Removes STL mesh files from
the earlier abandoned approach.

Co-Authored-By: Claude Sonnet 4.6 <noreply@anthropic.com>

File: so101_description/urdf/so101.urdf.xacro (robot description, xacro)
@@ -3,6 +3,4 @@
   <xacro:arg name="namespace" default=""/>
   <xacro:arg name="controllers_yaml" default="$(find so101_description)/config/ros2_controllers.yaml"/>
-  <!-- Set screwdriver:=true to add the screwdriver end-effector (used by screw_robot) -->
-  <xacro:arg name="screwdriver" default="false"/>
   <!-- Materials -->
   <material name="3d_printed">
@@ -350,51 +348,3 @@
     </plugin>
   </gazebo>
-  <!-- ============================================================
-       Screwdriver end-effector (enabled when screwdriver:=true)
-       Attaches to gripper_link; bit points in −Z of gripper_link frame.
-       Geometry (both STLs are in mm → scale 0.001):
-         bit_holder : 20mm ⌀ × 25.6mm tall, base at Z=0, tip at +Z in STL
-         screwdriver_bit : 4mm ⌀ × 43mm long
-       Both are flipped 180° (rpy π 0 0) so the tip extends in −Z.
-  ============================================================ -->
-  <xacro:if value="$(arg screwdriver)">
-    <link name="screwdriver_tip_link">
-      <inertial>
-        <origin xyz="0 0 -0.035" rpy="0 0 0"/>
-        <mass value="0.025"/>
-        <inertia ixx="1e-5" ixy="0" ixz="0" iyy="1e-5" iyz="0" izz="1e-6"/>
-      </inertial>
-      <!-- bit holder: flipped so chuck tip points in −Z -->
-      <visual>
-        <origin xyz="0 0 0" rpy="3.14159 0 0"/>
-        <geometry>
-          <mesh filename="package://so101_description/meshes/so101_screwdriver_bit_holder.stl"
-                scale="0.001 0.001 0.001"/>
-        </geometry>
-        <material name="sts3215"/>
-      </visual>
-      <!-- screwdriver bit: starts just below the holder tip -->
-      <visual>
-        <origin xyz="0 0 -0.026" rpy="3.14159 0 0"/>
-        <geometry>
-          <mesh filename="package://so101_description/meshes/screwdriver_bit.stl"
-                scale="0.001 0.001 0.001"/>
-        </geometry>
-        <material name="3d_printed"/>
-      </visual>
-      <!-- simplified collision: cylinder covering holder + bit -->
-      <collision>
-        <origin xyz="0 0 -0.035" rpy="0 0 0"/>
-        <geometry>
-          <cylinder radius="0.005" length="0.070"/>
-        </geometry>
-      </collision>
-    </link>
-    <!-- Fixed joint: 30mm below gripper_link origin, aligned with tool axis -->
-    <joint name="screwdriver_tip_joint" type="fixed">
-      <origin xyz="0 0 -0.030" rpy="0 0 0"/>
-      <parent link="gripper_link"/>
-      <child link="screwdriver_tip_link"/>
-    </joint>
-  </xacro:if>
 </robot>

File: so101_description/urdf/so101_screwdriver.urdf.xacro (robot description, xacro)
@@ -2,22 +2,82 @@
 <!--
   Screwdriver variant of the SO-101 arm.
-  Includes so101.urdf.xacro with screwdriver:=true, which adds:
-    - screwdriver_tip_link  (bit_holder mesh + screwdriver_bit mesh)
-    - screwdriver_tip_joint (fixed, parent gripper_link)
+  Includes so101.urdf.xacro unchanged, then conditionally appends a
+  2.5 mm hex screwdriver tip modelled from primitives:
+    - shaft   : cylinder r=4 mm, l=50 mm
+    - taper   : cylinder r=2 mm, l=5 mm
+    - hex bit : box 2.5×2.5×12 mm
+  The tip is attached as a fixed child of gripper_link pointing −Z.
   Usage (xacro.process_file):
-    mappings={'namespace': 'screw_robot'}          # screwdriver defaults to true
-    mappings={'namespace': 'screw_robot',
-              'screwdriver': 'false'}               # override to suppress tip
-  Pass namespace and controllers_yaml as usual — they flow through to
-  so101.urdf.xacro unchanged.
+    mappings={'namespace': 'screw_robot', 'screwdriver': 'true'}   # with tip
+    mappings={'namespace': 'some_arm'}                              # no tip (default false)
 -->
 <robot name="so101" xmlns:xacro="http://www.ros.org/wiki/xacro">
-  <!-- Declare args before the include so the screwdriver default is true.
-       xacro uses first-declaration-wins; the inner file's default="false"
-       for screwdriver is therefore a no-op. -->
+  <!-- Declare args before include so they are available to the inner file.
+       xacro uses first-declaration-wins; the inner file's own declarations
+       for namespace and controllers_yaml are therefore no-ops. -->
   <xacro:arg name="namespace"        default=""/>
   <xacro:arg name="controllers_yaml"
              default="$(find so101_description)/config/ros2_controllers.yaml"/>
-  <xacro:arg name="screwdriver"      default="true"/>
+  <xacro:arg name="screwdriver"      default="false"/>
   <xacro:include filename="$(find so101_description)/urdf/so101.urdf.xacro"/>
+  <!-- ── Screwdriver tip (only when screwdriver:=true) ─────────────────── -->
+  <xacro:if value="$(arg screwdriver)">
+    <link name="screwdriver_tip_link">
+      <inertial>
+        <!-- Centre of mass at mid-shaft -->
+        <origin xyz="0 0 -0.025" rpy="0 0 0"/>
+        <mass value="0.05"/>
+        <!-- Thin solid cylinder approx: ixx = iyy = m(3r²+l²)/12, izz = mr²/2
+             r=0.004 m  l=0.050 m  m=0.05 kg
+             ixx = 0.05*(3*0.000016+0.0025)/12 = 1.058e-5
+             izz = 0.05*0.000016/2             = 4.0e-7                      -->
+        <inertia ixx="1.06e-05" ixy="0" ixz="0"
+                 iyy="1.06e-05" iyz="0"
+                 izz="4.0e-07"/>
+      </inertial>
+      <!-- Shaft: cylinder r=4 mm, l=50 mm, centred at (0,0,-0.025) -->
+      <visual>
+        <origin xyz="0 0 -0.025" rpy="0 0 0"/>
+        <geometry>
+          <cylinder radius="0.004" length="0.050"/>
+        </geometry>
+        <material name="screwdriver_silver">
+          <color rgba="0.7 0.7 0.7 1.0"/>
+        </material>
+      </visual>
+      <!-- Taper: cylinder r=2 mm, l=5 mm, just below shaft tip -->
+      <visual>
+        <origin xyz="0 0 -0.0525" rpy="0 0 0"/>
+        <geometry>
+          <cylinder radius="0.002" length="0.005"/>
+        </geometry>
+        <material name="screwdriver_silver">
+          <color rgba="0.7 0.7 0.7 1.0"/>
+        </material>
+      </visual>
+      <!-- Hex bit: box 2.5×2.5×12 mm, below taper -->
+      <visual>
+        <origin xyz="0 0 -0.061" rpy="0 0 0"/>
+        <geometry>
+          <box size="0.0025 0.0025 0.012"/>
+        </geometry>
+        <material name="screwdriver_silver">
+          <color rgba="0.7 0.7 0.7 1.0"/>
+        </material>
+      </visual>
+      <!-- Collision: single cylinder encompassing shaft + taper + bit -->
+      <collision>
+        <origin xyz="0 0 -0.0335" rpy="0 0 0"/>
+        <geometry>
+          <cylinder radius="0.004" length="0.067"/>
+        </geometry>
+      </collision>
+    </link>
+    <joint name="screwdriver_tip_joint" type="fixed">
+      <!-- Offset 30 mm down from gripper_link origin along −Z -->
+      <origin xyz="0 0 -0.030" rpy="0 0 0"/>
+      <parent link="gripper_link"/>
+      <child  link="screwdriver_tip_link"/>
+    </joint>
+  </xacro:if>
 </robot>

Commit message: feat: step 2.6 — gripper with contact sensor and attach mechanism
- so101.urdf.xacro: add Gazebo contact sensor on moving_jaw link,
  topic scoped to /{namespace}/gripper/contact via xacro arg
- assembly_world.launch.py: replace single /gripper/contact bridge
  with per-arm entries; launch gripper_attach_node for all 4
  standard arms (not screw_robot) 2 s after arm controller up
- gripper_attach_node.py: Python node — monitors joint_states +
  contact topic, attaches screw to gripper tip via gz set_pose
  teleportation when gripper closes, releases on open
- CMakeLists.txt: install gripper_attach_node.py

Co-Authored-By: Claude Sonnet 4.6 <noreply@anthropic.com>

File: so101_description/urdf/so101.urdf.xacro (robot description, xacro)
@@ -348,3 +348,14 @@
     </plugin>
   </gazebo>
+  <!-- Contact sensor on moving jaw — per-arm gz topic via namespace arg -->
+  <gazebo reference="moving_jaw_so101_v1_link">
+    <sensor name="gripper_contact_sensor" type="contact">
+      <always_on>true</always_on>
+      <update_rate>100</update_rate>
+      <contact>
+        <collision>moving_jaw_so101_v1_link_collision</collision>
+      </contact>
+      <topic>$(arg namespace)/gripper/contact</topic>
+    </sensor>
+  </gazebo>
 </robot>
